File: Arduino_UNO_R3/UNO-TH_Rev3e.kicad_sch (KiCad schematic)
At the start: 116 parts, among them T1 FDN340P, U1 NCP1117ST50T3G, U2 LP2985-33DBVR, U3 ATMEGA16U2-MU(R), U5 LMV358IDGKR, X1 POWERSUPPLY_DC21MMX, X2 USB-B_TH, Y1 16MHz, Y2 CSTCE16M0V53-R0 16MHZ

Commit message: added datasheet and header details for R3
Parts:
- AD0: value 6x1F-H8.5 -> SSW-106-01-F-S
- IOH0: value 10x1F-H8.5 -> SSW-110-01-F-S
- IOL0: value 8x1F-H8.5 -> SSW-106-01-F-S
- POWER0: value 8x1F-H8.5 -> SSW-108-01-F-S
